File: weather_station/weather_station.kicad_sch (KiCad schematic)
At the start: 38 parts, among them J1 USB_C_Receptacle_USB2.0_16P, Q1 S8050, Q2 S8050, U2 AMS1117-3.3, U4 CP2102N-Axx-xQFN28

Commit message: Schematic done, Layout in progress
Parts:
- removed U2: AMS1117-3.3, Package_TO_SOT_SMD:SOT-223-3_TabPin2, symbol Regulator_Linear:AMS1117-3.3
- added C1, C14, C16, C18, C19, C5, C7: 100n, Capacitor_SMD:C_0603_1608Metric, symbol Device:C
- added C13, C15, C17: 22u, Capacitor_SMD:C_0805_2012Metric, symbol Device:C
- added C6: 10u, Capacitor_SMD:C_0805_2012Metric, symbol Device:C
- added D4, D5: LED, LED_SMD:LED_0603_1608Metric, symbol Device:LED
- added H1: MountingHole, weather_station_lib:mounting_hole_1.5, symbol Mechanical:MountingHole
- added L1: 2u2, weather_station_lib:Inductor_4.5x4.1x2, symbol Device:L
- added Q1: PMOS, weather_station_lib:SOT-23_(pins_inverted), symbol Simulation_SPICE:PMOS
- added R1, R10, R12, R14, R16, R17, R18: 1k, Resistor_SMD:R_0603_1608Metric_Pad0.98x0.95mm_HandSolder, symbol Device:R
- added R13, R15, R8: 100k, Resistor_SMD:R_0603_1608Metric_Pad0.98x0.95mm_HandSolder, symbol Device:R
- added R2, R7: 390k, Resistor_SMD:R_0603_1608Metric_Pad0.98x0.95mm_HandSolder, symbol Device:R
- added R5: 22k1, Resistor_SMD:R_0603_1608Metric_Pad0.98x0.95mm_HandSolder, symbol Device:R
- added R9: 12k, Resistor_SMD:R_0603_1608Metric_Pad0.98x0.95mm_HandSolder, symbol Device:R
- added SW1, SW2, SW3: SW_Push, weather_station_lib:tactile_switch_6x6, symbol weather_station_lib:SW_Push
- added TP6: TestPoint_2Pole, TestPoint:TestPoint_2Pads_Pitch5.08mm_Drill1.3mm, symbol Connector:TestPoint_2Pole
- added U2: TLV62569, Package_TO_SOT_SMD:SOT-23-5, symbol weather_station_lib:TLV62569DBVR
- added U3: TP4056-42-ESOP8, Package_SO:SOIC-8-1EP_3.9x4.9mm_P1.27mm_EP2.41x3.3mm_ThermalVias, symbol Battery_Management:TP4056-42-ESOP8
- added U5: Ai-Thinker-Ra-02, RF_Module:Ai-Thinker-Ra-01-LoRa, symbol RF_Module:Ai-Thinker-Ra-02
- added U6: ~, weather_station_lib:0.96inch_lcd, symbol weather_station_lib:0.96inch_lcd
- added X1: ~, weather_station_lib:Header_7x2.54_smt, symbol weather_station_lib:Header_7x2.54_smt
- C10: renamed from C3; footprint Capacitor_SMD:C_0805_2012Metric -> Capacitor_SMD:C_0603_1608Metric
- C11: renamed from C5; footprint Capacitor_SMD:C_0805_2012Metric -> Capacitor_SMD:C_0603_1608Metric
- C12: renamed from C6; footprint Capacitor_SMD:C_0805_2012Metric -> Capacitor_SMD:C_0603_1608Metric
- C4: renamed from C7; footprint Capacitor_SMD:C_0805_2012Metric -> Capacitor_SMD:C_0603_1608Metric
- C8: footprint Capacitor_SMD:C_0805_2012Metric -> Capacitor_SMD:C_0603_1608Metric
- C9: renamed from C4; footprint Capacitor_SMD:C_0805_2012Metric -> Capacitor_SMD:C_0603_1608Metric
- U4: renamed from U3; now not fitted
- U7: renamed from U4; now not fitted
- renumbered C1 to C3, D2 to D1, D1 to D2, D5 to D3, D3 to D6, D4 to D7, Q1 to Q2, Q2 to Q3, R4 to R11, R5 to R19, R10 to R20, R11 to R21, R7 to R22, R6 to R23, R12 to R24, R13 to R25, R8 to R26, R9 to R27, R2 to R4, R1 to R6, TP3 to TP1, TP4 to TP2, TP5 to TP3, TP1 to TP4, TP2 to TP5
Connections:
- net +Vch: now also C6.1, D4.2 (A), D5.2 (A), U3.4 (V_{CC}), U3.8 (CE)
- net +Vin: now also C2.1, C13.1, C14.1, C15.1, C16.1, C17.1, C18.1, C19.1, L1.2, R2.1, U5.3 (VDD), U6.2 (VDD), X1.2 (VDD); no longer D2.1 (K)
- net GND: now also TP1.1, U1.15 (GND), U1.38 (GND), U1.39 (GND), C1.2, C13.2, C14.2, C15.2, C16.2, C17.2, C18.2, C19.2, C5.2, C6.2, C7.2, R15.1, R18.1, R7.1, R8.1, R9.1, SW1.4 (A), SW2.4 (A), SW3.4 (A), TP6.2, U2.2 (GND), U3.1 (TEMP), U3.3 (GND), U3.9 (EPAD), U5.1 (GND), U5.16 (GND), U5.2 (GND), U5.9 (GND), U6.1 (GND), X1.1 (GND)
- net Vusb: now also D2.2 (A), Q1.2 (G), R9.2; no longer C3.1
- net VBAT_S: now reaches U1.10 (IO25)
- net VBAT_S: now also R13.1, R15.2
- net LORA_IRQ: now reaches U1.11 (IO26)
- net LORA_IRQ: now also U5.5 (DIO0)
- net LORA_RST: now reaches U1.12 (IO27)
- net LORA_RST: now also U5.4 (~{RESET})
- net SPI_CLK: now reaches U1.13 (IO14_HSPI_CLK)
- net SPI_CLK: now also U5.12 (SCK)
- net SPI_MISO: now reaches U1.14 (S_IO12_HSPI_MISO)
- net SPI_MISO: now also U5.13 (MISO)
- net SPI_MOSI: now reaches U1.16 (H_MOSI)
- net SPI_MOSI: now also U5.14 (MOSI)
- net SPI_CS: now reaches U1.23 (S_IO15_HCS)
- net SPI_CS: now also U5.15 (~{NSS})
- net BTN2: now reaches U1.26 (IO4)
- net BTN2: now also C7.1, R12.2
- net BTN1: now reaches U1.27 (IO16)
- net BTN1: now also C5.1, R10.2
- net TFT_RST: now reaches U1.28 (IO17)
- net TFT_RST: now also X1.5 (RES)
- net TFT_CS: now reaches U1.29 (S_IO5)
- net TFT_CLK: now reaches U1.30 (IO18)
- net TFT_CLK: now also X1.3 (SCL)
- net BTN0: now reaches U1.31 (IO19)
- net BTN0: now also C1.1, R1.2
- net TFT_SDA: now reaches U1.37 (IO23)
- net TFT_SDA: now also X1.4 (SDA)
- net SDA1: now reaches U1.6 (IO34)
- net SDA1: now also U6.4 (SDA)
- net SCL1: now reaches U1.7 (IO35)
- net SCL1: now also U6.3 (SCL)
- net TFT_BLK: now reaches U1.8 (IO32)
- net TFT_BLK: now also X1.7 (BLK)
- net TFT_DC: now reaches U1.9 (IO33)
- net TFT_DC: now also X1.6 (DC)
- removed net +3v3: C2.1, D2.2 (A)
- net SCL renamed SCL0
- net SDA renamed SDA0
- new net: R5.2, R8.2, U2.5 (FB)
- new net: D5.1 (K), R16.1
- new net: R12.1, SW3.1
- new net: R10.1, SW2.1
- new net: C3.1, D2.1 (K), Q1.3 (S), R7.2, U2.1 (EN), U2.4 (VIN)
- new net: R17.1, R18.2
- new net: D4.1 (K), R14.1
- new net: R17.2, U3.2 (PROG)
- new net: R16.2, U3.6 (~{STDBY})
- new net: R14.2, U3.7 (~{CHRG})
- new net: L1.1, U2.3 (SW)
- new net: R2.2, R5.1
- new net: R1.1, SW1.1
- new net +Vbat: Q1.1 (D), R13.2, TP6.1, U3.5 (BAT)
- no-connect marks 16 -> 37
Other:
- note added: "Has internal pullup on SDA and SCL"
- note added: "Vout = 3.07V"
- company: (none) -> Author: Erik Miyoshi
- title: (none) -> Wireless Weather Station
- moved on the sheet: C3, C4, C8, D1, D2, D3, J1, Q2, Q3, R11, R26, R27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

Commit message: Adjusting components
Parts:
- added H2, H3, H4: MountingHole, weather_station_lib:mounting_hole_2, symbol Mechanical:MountingHole
- C1, C11, C14, C16, C18, C19, C5, C7, C9: LCSC Part # (none) -> C14663; LCSCPN C14663 -> (none)
- C10, C12: LCSC Part # (none) -> C69335; LCSCPN C69335 -> (none)
- C13, C15, C17, C2: LCSC Part # (none) -> C602037; LCSCPN C602037 -> (none)
- C3, C6: LCSC Part # (none) -> C15850; LCSCPN C15850 -> (none)
- C4, C8: LCSC Part # (none) -> C100040; LCSCPN C100040 -> (none)
- D1, D2: LCSC Part # (none) -> C2986110; LCSCPN C2986110 -> (none)
- D3: LCSC Part # (none) -> C3040626; LCSCPN C3040626 -> (none)
- D4, D5, D6, D7: LCSC Part # (none) -> C965799; LCSCPN C965799 -> (none)
- H1: footprint weather_station_lib:mounting_hole_1.5 -> weather_station_lib:mounting_hole_2
- J1: footprint Connector_USB:USB_C_Receptacle_GCT_USB4105-xx-A_16P_TopMnt_Horizontal -> weather_station_lib:USB_C_Receptacle_GCT_USB4105-xx-A_16P_TopMnt_Horizontal_fix_clearance; LCSC Part # (none) -> C2765186; LCSCPN C2765186 -> (none)
- L1: LCSC Part # (none) -> C22463806; LCSCPN C22463806 -> (none)
- Q1: LCSC Part # (none) -> C2891731; LCSCPN C2891731 -> (none)
- Q2, Q3: LCSC Part # (none) -> C181158; LCSCPN C181158 -> (none)
- R1, R10, R12, R14, R16, R17, R18, R19, R24, R25: LCSC Part # (none) -> C22548; LCSCPN C22548 -> (none)
- R11, R26, R27, R3, R9: LCSC Part # (none) -> C114659; LCSCPN C114659 -> (none)
- R13, R15, R8: LCSC Part # (none) -> C14675; LCSCPN C14675 -> (none)
- R2, R7: LCSC Part # (none) -> C23150; LCSCPN C23150 -> (none)
- R20: LCSC Part # (none) -> C114669; LCSCPN C114669 -> (none)
- R21: LCSC Part # (none) -> C100044; LCSCPN C100044 -> (none)
- R22, R5: LCSC Part # (none) -> C137768; LCSCPN C137768 -> (none)
- R23: LCSC Part # (none) -> C2933225; LCSCPN C2933225 -> (none)
- R4, R6: LCSC Part # (none) -> C23186; LCSCPN C23186 -> (none)
- SW1, SW2, SW3: LCSC Part # (none) -> C455110; LCSCPN C455110 -> (none)
- TP1, TP2, TP3, TP4, TP5, TP6, U4, U6, U7, X1: now left out of the parts list
- U1: footprint weather_station_lib:ESP32-WROOM-32 or ESP32S -> weather_station_lib:ESP32-WROOM-32 or ESP32S_no_paste; now not fitted; now left out of the parts list
- U2: LCSC Part # (none) -> C141836; LCSCPN C141836 -> (none)
- U3: LCSC Part # (none) -> C725790; LCSCPN C725790 -> (none)
- U5: footprint RF_Module:Ai-Thinker-Ra-01-LoRa -> weather_station_lib:Ai-Thinker-Ra-01-LoRa_no_paste; now left out of the parts list
Connections:
- net +Vin: now also U6.3 (VDD); no longer U6.2 (VDD)
- net GND: now also U6.4 (GND); no longer U6.1 (GND)
- net SCL1: now also U6.2 (SCL); no longer U6.3 (SCL)
- net SDA1: now also U6.1 (SDA); no longer U6.4 (SDA)
Other:
- moved on the sheet: H1

Commit message: Adjust min via hole size to 0.3mm
Parts:
- C1, C11, C14, C16, C18, C19, C5, C7, C9: Voltage 25V -> 50V
- C10, C12: footprint Capacitor_SMD:C_0603_1608Metric -> Capacitor_SMD:C_0805_2012Metric; LCSC Page https://www.lcsc.com/product-detail/Multilayer-Ceramic-Capacitors-MLCC-SMD-SMT_Samsung-Electro-Mechanics-CL10A475KA8NQNC_C69335.html -> https://www.lcsc.com/product-detail/Multilayer-Ceramic-Capacitors-MLCC-SMD-SMT_Samsung-Electro-Mechanics-CL21A475KAQNNNE_C1779.html?s_z=n_%2520C1779; LCSC Part # C69335 -> C1779
- C13, C15, C17, C2: LCSC Page https://www.lcsc.com/product-detail/Multilayer-Ceramic-Capacitors-MLCC-SMD-SMT_Samsung-Electro-Mechanics-CL21A226MAYNNNE_C602037.html -> https://www.lcsc.com/product-detail/Multilayer-Ceramic-Capacitors-MLCC-SMD-SMT_Samsung-Electro-Mechanics-CL21A226MAQNNNE_C45783.html?s_z=n_%2520C45783; LCSC Part # C602037 -> C45783
- C4, C8: LCSC Page https://www.lcsc.com/product-detail/Multilayer-Ceramic-Capacitors-MLCC-SMD-SMT_YAGEO-CC0603KRX7R9BB102_C100040.html -> https://www.lcsc.com/product-detail/Multilayer-Ceramic-Capacitors-MLCC-SMD-SMT_Samsung-Electro-Mechanics-CL10B102KB8NNNC_C1588.html?s_z=n_%2520C1588; LCSC Part # C100040 -> C1588; Voltage 25V -> 50V
- D1, D2: LCSC Page https://www.lcsc.com/product-detail/Schottky-Diodes_GOODWOR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 -> https://www.lcsc.com/product-detail/Schottky-Diodes_MDD-Mic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; LCSC Part # C2986110 -> C2480
- D4, D5, D6, D7: LCSC Page https://www.lcsc.com/product-detail/LED-Indication-Discrete_XINGLIGHT-XL-1608SURC-06_C965799.html -> https://www.lcsc.com/product-detail/LED-Indication-Discrete_Hubei-KENTO-Elec-KT-0603R_C2286.html?s_z=n_%2520C2286; LCSC Part # C965799 -> C2286
- Q1: LCSC Page https://www.lcsc.com/product-detail/MOSFETs_YONGYUTAI-SI230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 -> https://www.lcsc.com/product-detail/MOSFETs_Alpha-Omega-Sem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; LCSC Part # C2891731 -> C15127; PN SI2301 -> AO3401A
- Q2, Q3: value S8050 -> MMBT3904; LCSC Page https://www.lcsc.com/product-detail/Bipolar-BJT_Guangdong-H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 -> https://www.lcsc.com/product-detail/Bipolar-BJT_Jiangsu-Cha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; LCSC Part # C181158 -> C20526
- R1, R10, R12, R14, R16, R17, R18, R19, R24, R25: LCSC Page https://www.lcsc.com/product-detail/Chip-Resistor-Surface-Mount_YAGEO-RC0603FR-071KL_C22548.html -> https://www.lcsc.com/product-detail/Chip-Resistor-Surface-Mount_UNI-ROYAL-Uniroyal-Elec-0603WAF1001T5E_C21190.html?s_z=n_C21190; LCSC Part # C22548 -> C21190
- R11, R26, R27, R3, R9: LCSC Page https://www.lcsc.com/product-detail/Chip-Resistor-Surface-Mount_YAGEO-RC0603FR-0712KL_C114659.html -> https://www.lcsc.com/product-detail/Chip-Resistor-Surface-Mount_UNI-ROYAL-Uniroyal-Elec-0603WAF1202T5E_C22790.html?s_z=n_C22790; LCSC Part # C114659 -> C22790
- R13, R15, R8: LCSC Page https://www.lcsc.com/product-detail/Chip-Resistor-Surface-Mount_YAGEO-RC0603FR-07100KL_C14675.html -> https://www.lcsc.com/product-detail/Chip-Resistor-Surface-Mount_UNI-ROYAL-Uniroyal-Elec-0603WAF1003T5E_C25803.html?s_z=n_C25803; LCSC Part # C14675 -> C25803
- R2, R7: value 390k -> 470k; LCSC Page https://www.lcsc.com/product-detail/Chip-Resistor-Surface-Mount_UNI-ROYAL-Uniroyal-Elec-0603WAF3903T5E_C23150.html -> https://www.lcsc.com/product-detail/Chip-Resistor-Surface-Mount_UNI-ROYAL-Uniroyal-Elec-0603WAF4703T5E_C23178.html?s_z=n_C23178; LCSC Part # C23150 -> C23178
- R20: LCSC Page https://www.lcsc.com/product-detail/Chip-Resistor-Surface-Mount_YAGEO-RC0603FR-07470RL_C114669.html -> https://www.lcsc.com/product-detail/Chip-Resistor-Surface-Mount_UNI-ROYAL-Uniroyal-Elec-0603WAF4700T5E_C23179.html?s_z=n_C23179; LCSC Part # C114669 -> C23179
- R21: LCSC Page https://www.lcsc.com/product-detail/Chip-Resistor-Surface-Mount_YAGEO-RC0603FR-070RL_C100044.html -> https://www.lcsc.com/product-detail/Chip-Resistor-Surface-Mount_UNI-ROYAL-Uniroyal-Elec-0603WAF0000T5E_C21189.html?s_z=n_C21189; LCSC Part # C100044 -> C21189
- R22: value 22k1 -> 22k; LCSC Page https://www.lcsc.com/product-detail/Chip-Resistor-Surface-Mount_YAGEO-RC0603FR-0722K1L_C137768.html -> https://www.lcsc.com/product-detail/Chip-Resistor-Surface-Mount_UNI-ROYAL-Uniroyal-Elec-0603WAF2202T5E_C31850.html?s_z=n_C31850; LCSC Part # C137768 -> C31850
- R23: value 47k5 -> 47k; LCSC Page https://www.lcsc.com/product-detail/Chip-Resistor-Surface-Mount_FOJAN-FRC0603F4752TS_C2933225.html -> https://www.lcsc.com/product-detail/Chip-Resistor-Surface-Mount_UNI-ROYAL-Uniroyal-Elec-0603WAF4702T5E_C25819.html?s_z=n_C25819; LCSC Part # C2933225 -> C25819
- R4, R6: LCSC Page https://www.lcsc.com/product-detail/Chip-Resistor-Surface-Mount_UNI-ROYAL-Uniroyal-Elec-0603WAF5101T5E_C23186.html -> https://www.lcsc.com/product-detail/Chip-Resistor-Surface-Mount_UNI-ROYAL-Uniroyal-Elec-0603WAF5101T5E_C23186.html?s_z=n_C23186
- R5: value 22k1 -> 12k; LCSC Page https://www.lcsc.com/product-detail/Chip-Resistor-Surface-Mount_YAGEO-RC0603FR-0722K1L_C137768.html -> https://www.lcsc.com/product-detail/Chip-Resistor-Surface-Mount_UNI-ROYAL-Uniroyal-Elec-0603WAF1202T5E_C22790.html?s_z=n_C22790; LCSC Part # C137768 -> C22790
- U3: footprint Package_SO:SOIC-8-1EP_3.9x4.9mm_P1.27mm_EP2.41x3.3mm_ThermalVias -> weather_station_lib:SOIC-8-1EP_3.9x4.9mm_P1.27mm_EP2.41x3.3mm_ThermalVias_via_0.3mm
- U7: footprint Package_DFN_QFN:QFN-28-1EP_5x5mm_P0.5mm_EP2.7x2.7mm_ThermalVias -> weather_station_lib:QFN-28-1EP_5x5mm_P0.5mm_EP2.7x2.7mm_ThermalVias_via_0.3mm
Connections:
- net at R5.2, U2.5 (FB): now also R2.2; no longer R8.2
- net at R5.1: now also R8.2; no longer R2.2
Other:
- note added: "Vout = 3.12V"
- note removed: "Vout = 3.07V"
