File: HW/weather_station/weather_station.kicad_sch (KiCad schematic)
At the start: 79 parts, among them J1 USB_C_Receptacle_USB2.0_16P, Q1 PMOS, Q2 MMBT3904, Q3 MMBT3904, SW1 SW_Push, SW2 SW_Push, SW3 SW_Push, U2 TLV62569, U3 TP4056-42-ESOP8, U5 Ai-Thinker-Ra-02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

Commit message: Generating pdf files for hw
Parts:
- U1: now fitted; now in the parts list
- U4, U5, U6: now fitted
Changed lines of the file:
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@@
 		(in_bom no)
 		(on_board yes)
-		(dnp yes)
+		(dnp no)
 		(property "Reference" "U4"
 			(at 266.7 120.396 0)
@@
 		(unit 1)
 		(exclude_from_sim no)
-		(in_bom no)
+		(in_bom yes)
 		(on_board yes)
-		(dnp yes)
+		(dnp no)
 		(fields_autoplaced yes)
 		(property "Reference" "U1"
@@
 		(in_bom no)
 		(on_board yes)
-		(dnp yes)
+		(dnp no)
 		(fields_autoplaced yes)
 		(property "Reference" "U6"
@@
 		(in_bom no)
 		(on_board yes)
-		(dnp yes)
+		(dnp no)
 		(fields_autoplaced yes)
 		(property "Reference" "U5"
